Commit message: modify solo files

File: files/solo_description/solo12.urdf (robot description, URDF)
Before this commit: robot solo, 17 links, 16 joints
Links:
- link FL_LOWER_LEG: geometry collision mesh filename=/home/khorshidi/git/system_identification/files/solo_descri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; visual mesh filename=/home/khorshidi/git/system_identification/files/solo_descri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
- link FL_SHOULDER: geometry collision mesh filename=/home/khorshidi/git/system_identification/files/solo_descri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; visual mesh filename=/home/khorshidi/git/system_identification/files/solo_descri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
- link FL_UPPER_LEG: geometry collision mesh filename=/home/khorshidi/git/system_identification/files/solo_descri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; visual mesh filename=/home/khorshidi/git/system_identification/files/solo_descri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
- link FR_LOWER_LEG: geometry collision mesh filename=/home/khorshidi/git/system_identification/files/solo_descri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; visual mesh filename=/home/khorshidi/git/system_identification/files/solo_descri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
- link FR_SHOULDER: geometry collision mesh filename=/home/khorshidi/git/system_identification/files/solo_descri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; visual mesh filename=/home/khorshidi/git/system_identification/files/solo_descri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
- link FR_UPPER_LEG: geometry collision mesh filename=/home/khorshidi/git/system_identification/files/solo_descri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; visual mesh filename=/home/khorshidi/git/system_identification/files/solo_descri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
- link HL_LOWER_LEG: geometry collision mesh filename=/home/khorshidi/git/system_identification/files/solo_descri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; visual mesh filename=/home/khorshidi/git/system_identification/files/solo_descri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
- link HL_SHOULDER: geometry collision mesh filename=/home/khorshidi/git/system_identification/files/solo_descri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; visual mesh filename=/home/khorshidi/git/system_identification/files/solo_descri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
- link HL_UPPER_LEG: geometry collision mesh filename=/home/khorshidi/git/system_identification/files/solo_descri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; visual mesh filename=/home/khorshidi/git/system_identification/files/solo_descri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
- link HR_LOWER_LEG: geometry collision mesh filename=/home/khorshidi/git/system_identification/files/solo_descri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; visual mesh filename=/home/khorshidi/git/system_identification/files/solo_descri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
- link HR_SHOULDER: geometry collision mesh filename=/home/khorshidi/git/system_identification/files/solo_descri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; visual mesh filename=/home/khorshidi/git/system_identification/files/solo_descri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
- link HR_UPPER_LEG: geometry collision mesh filename=/home/khorshidi/git/system_identification/files/solo_descri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; visual mesh filename=/home/khorshidi/git/system_identification/files/solo_descri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
- link base_link: geometry collision mesh filename=/home/khorshidi/git/system_identification/files/solo_descri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; visual mesh filename=/home/khorshidi/git/system_identification/files/solo_descri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

Commit message: modify solo files

File: files/solo_description/solo12.urdf (robot description, URDF)
Before this commit: robot solo, 17 links, 16 joints
Links:
- link FL_LOWER_LEG: geometry collision mesh filename=package://solo_description/mesh/stl/without_foot/solo_lower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; visual mesh filename=package://solo_description/mesh/stl/without_foot/solo_lower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
- link FL_SHOULDER: geometry collision mesh filename=package://solo_description/mesh/stl/solo12/solo12_hip_fe_fl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; visual mesh filename=package://solo_description/mesh/stl/solo12/solo12_hip_fe_fl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
- link FL_UPPER_LEG: geometry collision mesh filename=package://solo_description/mesh/stl/without_foot/solo_upper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; visual mesh filename=package://solo_description/mesh/stl/without_foot/solo_upper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
- link FR_LOWER_LEG: geometry collision mesh filename=package://solo_description/mesh/stl/without_foot/solo_lower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; visual mesh filename=package://solo_description/mesh/stl/without_foot/solo_lower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
- link FR_SHOULDER: geometry collision mesh filename=package://solo_description/mesh/stl/solo12/solo12_hip_fe_fr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; visual mesh filename=package://solo_description/mesh/stl/solo12/solo12_hip_fe_fr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
- link FR_UPPER_LEG: geometry collision mesh filename=package://solo_description/mesh/stl/without_foot/solo_upper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; visual mesh filename=package://solo_description/mesh/stl/without_foot/solo_upper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
- link HL_LOWER_LEG: geometry collision mesh filename=package://solo_description/mesh/stl/without_foot/solo_lower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; visual mesh filename=package://solo_description/mesh/stl/without_foot/solo_lower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
- link HL_SHOULDER: geometry collision mesh filename=package://solo_description/mesh/stl/solo12/solo12_hip_fe_hl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; visual mesh filename=package://solo_description/mesh/stl/solo12/solo12_hip_fe_hl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
- link HL_UPPER_LEG: geometry collision mesh filename=package://solo_description/mesh/stl/without_foot/solo_upper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; visual mesh filename=package://solo_description/mesh/stl/without_foot/solo_upper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
- link HR_LOWER_LEG: geometry collision mesh filename=package://solo_description/mesh/stl/without_foot/solo_lower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; visual mesh filename=package://solo_description/mesh/stl/without_foot/solo_lower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
- link HR_SHOULDER: geometry collision mesh filename=package://solo_description/mesh/stl/solo12/solo12_hip_fe_hr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; visual mesh filename=package://solo_description/mesh/stl/solo12/solo12_hip_fe_hr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
- link HR_UPPER_LEG: geometry collision mesh filename=package://solo_description/mesh/stl/without_foot/solo_upper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; visual mesh filename=package://solo_description/mesh/stl/without_foot/solo_upper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
- link base_link: geometry collision mesh filename=package://solo_description/mesh/stl/solo12/solo_12_base.stl; visual mesh filename=package://solo_description/mesh/stl/solo12/solo_12_base.stl
