Commit message: modify spot files

File: files/spot_description/spot.urdf (robot description, URDF)
Before this commit: robot spot, 20 links, 19 joints
Links:
- removed link front_left_foot
- removed link front_right_foot
- removed link rear_left_foot
- removed link rear_right_foot
- added link fl_foot, mass 0.0
- added link fr_foot, mass 0.0
- added link rl_foot, mass 0.0
- added link rr_foot, mass 0.0
- link base_link: mass 32.86 -> 16.52; geometry visual mesh filename=package://spot_description/meshes/base/visual/body.obj
Joints:
- removed joint front_left_ankle
- removed joint front_right_ankle
- removed joint rear_left_ankle
- removed joint rear_right_ankle
- added joint fl_ankle: type fixed, parent front_left_lower_leg, child fl_foot, origin xyz=0 0 -0.35 rpy=0 0 0, limit lower=-10 upper=10 effort=1000 velocity=1000
- added joint fr_ankle: type fixed, parent front_right_lower_leg, child fr_foot, origin xyz=0 0 -0.35 rpy=0 0 0, limit lower=-10 upper=10 effort=1000 velocity=1000
- added joint rl_ankle: type fixed, parent rear_left_lower_leg, child rl_foot, origin xyz=0 0 -0.35 rpy=0 0 0, limit lower=-10 upper=10 effort=1000 velocity=1000
- added joint rr_ankle: type fixed, parent rear_right_lower_leg, child rr_foot, origin xyz=0 0 -0.35 rpy=0 0 0, limit lower=-10 upper=10 effort=1000 velocity=1000
